Commit message: Velodyne a funcionar
Signed-off-by: protobella <marianaleucadio@gmail.com>

File: sjtu-drone/urdf/sjtu_drone.urdf.xacro (robot description, xacro)
@@ -1,4 +1,8 @@
 <?xml version="1.0" ?>
-<robot name="sjtu_drone">
+<robot xmlns:xacro="http://www.ros.org/wiki/xacro" name="sjtu_drone">
+  <xacro:arg name="gpu" default="false"/>
+  <xacro:property name="gpu" value="$(arg gpu)" />
+  <xacro:arg name="organize_cloud" default="false"/>
+  <xacro:property name="organize_cloud" value="$(arg organize_cloud)" />
   <link name="base_link">
     <inertial>
@@ -7,5 +11,5 @@
       <inertia ixx="0.1152" ixy="0" ixz="0" iyy="0.1152" iyz="0" izz="0.218"/>
     </inertial>
-    <collision name="sjtu_drone__collision">
+    <collision name="sjtu_drone_collision">
       <origin rpy="0 0 0" xyz="0   0   0.04"/>
       <geometry>
@@ -85,54 +89,4 @@
         </sonar>
       </sensor>
-      <!-- Laser sensor -->
-      <sensor type="gpu_ray" name="velodyne-HDL32E">
-        <pose>0 0 0 0 0 0</pose>
-        <visualize>true</visualize>
-        <update_rate>10</update_rate>
-        <ray>
-          <scan>
-            <!-- Set horizontal FOV by setting image height -->
-            <!-- 512 beams with 90 degrees horizontal FOV (M900-90) -->
-            <horizontal>
-              <samples>512</samples>
-              <resolution>1</resolution>
-              <min_angle>-3.14</min_angle>
-              <max_angle>3.14</max_angle>
-            </horizontal>
-            <!-- Set vertical FOV by setting image height -->
-            <!-- Approx 2 times the spec sheet (sepc: 20 deg.) -->
-            <vertical>
-              <samples>300</samples>
-              <resolution>1</resolution>
-              <min_angle>-0.535</min_angle>
-              <max_angle>0.183</max_angle>
-            </vertical>
-          </scan>
-          <range>
-            <!-- min range is a collision range no need to change-->
-            <min>0.1</min>
-            <max>10.0</max>
-            <resolution>0.1</resolution>
-          </range>
-          <noise>
-            <type>gaussian</type>
-            <!-- Noise parameters based on published spec for Hokuyo laser
-                achieving "+-30mm" accuracy at range < 10m.  A mean of 0.0m and
-                stddev of 0.01m will put 99.7% of samples within 0.03m of the true
-                reading. -->
-            <mean>0.0</mean>
-            <stddev>0.01</stddev>
-          </noise>
-        </ray>
-        <plugin name="ray_sonar_sensor" filename="libgazebo_ros_velodyne_gpu_laser.so">
-          <topicName>/velodyne_points</topicName>
-          <frameName>velodyne</frameName>
-          <static_reference_frame>base_link</static_reference_frame>
-          <organize_cloud>true</organize_cloud>
-          <min_range>0.2</min_range>
-          <max_range>10.0</max_range>
-          <gaussianNoise>0.008</gaussianNoise>
-        </plugin>
-      </sensor>
     <!-- front camera -->
     <sensor name="front_camera" type="camera">
@@ -190,3 +144,8 @@
     </sensor>
   </gazebo>
+  <!-- Laser sensor -->
+  <xacro:include filename="$(find sjtu_drone)/urdf/velodyne.xacro"/>
+  <xacro:HDL-32E parent="base_link" name="velodyne" topic="/velodyne_points" organize_cloud="${organize_cloud}" hz="10" samples="220" gpu="${gpu}">
+    <origin xyz="0 0 0.04" rpy="0 0 0" />
+  </xacro:HDL-32E>
 </robot>

Commit message: Retificação da configuração rviz
Signed-off-by: protobella <marianaleucadio@gmail.com>

File: sjtu-drone/urdf/sjtu_drone.urdf.xacro (robot description, xacro)
@@ -108,5 +108,5 @@
         </noise>
       </camera>
-	    <pose> 0.2 0.0 0.0 0 0 0 </pose>
+	    <pose> 0.0 0.0 0.2 0 0 0 </pose>
       <always_on>1</always_on>
       <update_rate>60</update_rate>
@@ -147,5 +147,5 @@
   <xacro:include filename="$(find sjtu_drone)/urdf/velodyne.xacro"/>
   <xacro:HDL-32E parent="base_link" name="velodyne" topic="/velodyne_points" organize_cloud="${organize_cloud}" hz="10" samples="220" gpu="${gpu}">
-    <origin xyz="0 0 0.04" rpy="0 0 0" />
+    <origin xyz="0 0 0.1" rpy="0 0 0" />
   </xacro:HDL-32E>
 </robot>

Commit message: Colocar o sensor lidar na parte de baixo do drone
Signed-off-by: protobella <marianaleucadio@gmail.com>

File: sjtu-drone/urdf/sjtu_drone.urdf.xacro (robot description, xacro)
@@ -12,5 +12,5 @@
     </inertial>
     <collision name="sjtu_drone_collision">
-      <origin rpy="0 0 0" xyz="0   0   0.04"/>
+      <origin rpy="0 0 0" xyz="0   0   0.26"/>
       <geometry>
         <mesh filename="package://sjtu_drone/meshes/quadrotor_4.stl"/>
@@ -18,5 +18,5 @@
     </collision>
     <visual name="sjtu_drone__visual">
-      <origin rpy="0 0 0" xyz="0   0   0.04"/>
+      <origin rpy="0 0 0" xyz="0   0   0.26"/>
       <geometry>
         <mesh filename="package://sjtu_drone/meshes/quadrotor_4.dae"/>
@@ -55,5 +55,5 @@
   <!-- Sensors -->
   <gazebo reference="base_link">
-    	<sensor name='sensor_imu' type='imu'>
+    	<!-- <sensor name='sensor_imu' type='imu'>
         <always_on> 1 </always_on>
         <update_rate> 100 </update_rate>
@@ -74,7 +74,7 @@
           </noise>
         </imu>
-      </sensor>
+      </sensor> -->
       <!-- Sonar sensor in 100fps -->
-      <sensor name='sensor_sonar' type='sonar'>
+      <!-- <sensor name='sensor_sonar' type='sonar'>
         <always_on>1</always_on>
         <visualize>0</visualize>
@@ -88,5 +88,5 @@
           <radius>1.33974596</radius>
         </sonar>
-      </sensor>
+      </sensor> -->
     <!-- front camera -->
     <sensor name="front_camera" type="camera">
@@ -108,5 +108,5 @@
         </noise>
       </camera>
-	    <pose> 0.0 0.0 0.2 0 0 0 </pose>
+	    <pose> 0.0 0.0 0.6 0 0 0 </pose>
       <always_on>1</always_on>
       <update_rate>60</update_rate>
@@ -117,5 +117,5 @@
     </sensor>
 	  <!-- downward looking camera -->
-    <sensor name="down_camera" type="camera">
+    <!-- <sensor name="down_camera" type="camera">
       <camera>
         <horizontal_fov>1.047</horizontal_fov>
@@ -142,5 +142,5 @@
         <imageTopicName>/drone/down_camera/image_raw</imageTopicName>
       </plugin>
-    </sensor>
+    </sensor> -->
   </gazebo>
   <!-- Laser sensor -->

File: sjtu-drone/urdf/velodyne.xacro (robot description, xacro)
@@ -11,5 +11,5 @@
       <inertial>
         <mass value="1.0"/>
-        <origin xyz="0 0 0.07212"/>
+        <origin xyz="0 0 -0.07212"/>
         <inertia ixx="${(1.0 * (3.0*0.04267*0.04267 + 0.14424*0.14424)) / 12.0}" ixy="0" ixz="0"
           iyy="${(1.0 * (3.0*0.04267*0.04267 + 0.14424*0.14424)) / 12.0}" iyz="0"
@@ -22,5 +22,5 @@
       </visual>
       <collision>
-        <origin rpy="0 0 0" xyz="0 0 0.07212"/>
+        <origin rpy="0 0 0" xyz="0 0 -0.07212"/>
         <geometry>
           <cylinder radius="0.04267" length="0.14424"/>
